Commit message: Add files via upload

File: priv2/src/priv2_description/urdf/priv2.xacro (robot description, xacro)
@@ -7,5 +7,5 @@
     <inertial>
       <origin
-        xyz="0 0 0"
+        xyz="-0.025 0 0"
         rpy="0 0 0" />
       <mass      value="0.5" />
@@ -80,4 +80,6 @@
       </geometry>
     </collision>
+ <dynamics
+      friction="0.5" />
   </link>
    <joint
@@ -132,4 +134,6 @@
       </geometry>
     </collision>
+ <dynamics
+      friction="0.5" />
   </link>
   <joint
@@ -146,3 +150,152 @@
       xyz="0 0 -1" />
   </joint>
+  <!--<link   name="wheel_b">
+    <inertial>
+      <origin
+        xyz="0.00083781 -2.0474E-07 -2.0688E-07"
+        rpy="0 0 0" />
+      <mass
+        value="0.01" />
+      <inertia
+        ixx="4.3881E-08"
+        ixy="0"
+        ixz="0"
+        iyy="5.0048E-08"
+        iyz="0"
+        izz="5.0048E-08" />
+    </inertial>
+    <visual>
+      <origin
+        xyz="0 0 0"
+        rpy="0 0 0" />
+      <geometry>
+        <mesh
+          filename="package://priv2/src/priv2_description/meshes/wheel_b.STL" />
+      </geometry>
+      <material
+        name="">
+        <color
+          rgba="0.79216 0.81961 0.93333 1" />
+      </material>
+    </visual>
+    <collision>
+      <origin
+        xyz="0 0 0"
+        rpy="0 0 0" />
+      <geometry>
+        <mesh
+          filename="package://priv2/src/priv2_description/meshes/wheel_b.STL" />
+      </geometry>
+    </collision>
+  </link> -->
+ <link
+    name="wheel_b_axis">
+    <inertial>
+      <origin
+        xyz="-3.4694E-18 -0.0035 -1.7347E-18"
+        rpy="0 0 0" />
+      <mass
+        value="0.05" />
+      <inertia
+        ixx="2.7941E-08"
+        ixy="0"
+        ixz="0"
+        iyy="4.6383E-08"
+        iyz="0"
+        izz="2.3027E-08" />
+    </inertial>
+    <visual>
+      <origin
+        xyz="0 0 0"
+        rpy="0 0 0" />
+      <geometry>
+        <mesh
+          filename="package://priv2/src/priv2_description/meshes/wheel_b_axis.STL" />
+      </geometry>
+      <material
+        name="">
+        <color
+          rgba="0.79216 0.81961 0.93333 1" />
+      </material>
+    </visual>
+    <collision>
+      <origin
+        xyz="0 0 0"
+        rpy="0 0 0" />
+      <geometry>
+        <mesh
+          filename="package://priv2/src/priv2_description/meshes/wheel_b_axis.STL" />
+      </geometry>
+    </collision>
+<dynamics
+      friction="0.2" />
+  </link>
+  <joint
+    name="Joint_wheel_b"
+    type="continuous">
+    <origin
+      xyz="0.025024 -4.1596E-05 0.002"
+      rpy="-1.5708 0 2.5198" />
+    <parent
+      link="base_link" />
+    <child
+      link="wheel_b_axis" />
+    <axis
+      xyz="0 1 0" />
+    <dynamics
+      friction="0.002" />
+  </joint>
+  <link
+    name="wheel_b">
+    <inertial>
+      <origin
+        xyz="0 0 0"
+        rpy="0 0 0" />
+      <mass
+        value="0.05" />
+      <inertia
+        ixx="4.3881E-08"
+        ixy="0"
+        ixz="0"
+        iyy="5.0048E-08"
+        iyz="0"
+        izz="5.0048E-08" />
+    </inertial>
+    <visual>
+      <origin
+        xyz="0 0 0"
+        rpy="0 0 0" />
+      <geometry>
+        <mesh
+          filename="package://priv2/src/priv2_description/meshes/wheel_b.STL" />
+      </geometry>
+      <material
+        name="">
+        <color
+          rgba="0.79216 0.81961 0.93333 1" />
+      </material>
+    </visual>
+    <collision>
+      <origin
+        xyz="0 0 0"
+        rpy="0 0 0" />
+      <geometry>
+        <mesh
+          filename="package://priv2/src/priv2_description/meshes/wheel_b.STL" />
+      </geometry>
+    </collision>
+  </link>
+  <joint
+    name="Joint_wheel_b_axis"
+    type="continuous">
+    <origin
+      xyz="0 0 0"
+      rpy="-2.7485 0.94901 0" />
+    <parent
+      link="wheel_b_axis" />
+    <child
+      link="wheel_b" />
+    <axis
+      xyz="1 0 0" />
+  </joint>
 </robot>

Commit message: Add files via upload

File: priv2/src/priv2_description/urdf/priv2.xacro (robot description, xacro)
@@ -9,12 +9,12 @@
         xyz="-0.025 0 0"
         rpy="0 0 0" />
-      <mass      value="0.5" />
-      <inertia
-        ixx="4.38E-06"
-        ixy="0"
-        ixz="0"
-        iyy="5.67E-06"
-        iyz="0"
-        izz="2.17E-06" />
+      <mass      value="1" />
+      <inertia
+        ixx="0.000966667"
+        ixy="0"
+        ixz="0"
+        iyy="0.001133333"
+        iyz="0"
+        izz="0.000433333" />
     </inertial>
     <visual>
@@ -48,12 +48,12 @@
         rpy="0 0 0" />
       <mass
-        value="0.1" />
-      <inertia
-        ixx="1.08E-05"
-        ixy="0"
-        ixz="0"
-        iyy="1.08333E-05"
-        iyz="0"
-        izz="0.000001" />
+        value="0.5" />
+      <inertia
+        ixx="5.42E-05"
+        ixy="0"
+        ixz="0"
+        iyy="5.42E-05"
+        iyz="0"
+        izz="0.0001" />
     </inertial>
     <visual>
@@ -81,5 +81,5 @@
     </collision>
  <dynamics
-      friction="0.5" />
+      friction="1.4" />
   </link>
    <joint
@@ -102,12 +102,12 @@
         rpy="0 0 0" />
       <mass
-        value="0.1" />
-      <inertia
-        ixx="1.08E-05"
-        ixy="0"
-        ixz="0"
-        iyy="1.08333E-05"
-        iyz="0"
-        izz="0.000001" />
+        value="0.5" />
+      <inertia
+        ixx="5.42E-05"
+        ixy="0"
+        ixz="0"
+        iyy="5.42E-05"
+        iyz="0"
+        izz="0.0001" />
     </inertial>
     <visual>
@@ -135,5 +135,5 @@
     </collision>
  <dynamics
-      friction="0.5" />
+      friction="1.4" />
   </link>
   <joint
@@ -148,45 +148,6 @@
       link="wheel_l" />
     <axis
-      xyz="0 0 -1" />
-  </joint>
-  <!--<link   name="wheel_b">
-    <inertial>
-      <origin
-        xyz="0.00083781 -2.0474E-07 -2.0688E-07"
-        rpy="0 0 0" />
-      <mass
-        value="0.01" />
-      <inertia
-        ixx="4.3881E-08"
-        ixy="0"
-        ixz="0"
-        iyy="5.0048E-08"
-        iyz="0"
-        izz="5.0048E-08" />
-    </inertial>
-    <visual>
-      <origin
-        xyz="0 0 0"
-        rpy="0 0 0" />
-      <geometry>
-        <mesh
-          filename="package://priv2/src/priv2_description/meshes/wheel_b.STL" />
-      </geometry>
-      <material
-        name="">
-        <color
-          rgba="0.79216 0.81961 0.93333 1" />
-      </material>
-    </visual>
-    <collision>
-      <origin
-        xyz="0 0 0"
-        rpy="0 0 0" />
-      <geometry>
-        <mesh
-          filename="package://priv2/src/priv2_description/meshes/wheel_b.STL" />
-      </geometry>
-    </collision>
-  </link> -->
+      xyz="0 0 1" />
+  </joint>
  <link
     name="wheel_b_axis">
@@ -196,5 +157,5 @@
         rpy="0 0 0" />
       <mass
-        value="0.05" />
+        value="0.5" />
       <inertia
         ixx="2.7941E-08"
@@ -211,23 +172,21 @@
       <geometry>
         <mesh
-          filename="package://priv2/src/priv2_description/meshes/wheel_b_axis.STL" />
-      </geometry>
-      <material
-        name="">
-        <color
-          rgba="0.79216 0.81961 0.93333 1" />
-      </material>
-    </visual>
-    <collision>
-      <origin
-        xyz="0 0 0"
-        rpy="0 0 0" />
-      <geometry>
-        <mesh
-          filename="package://priv2/src/priv2_description/meshes/wheel_b_axis.STL" />
-      </geometry>
-    </collision>
-<dynamics
-      friction="0.2" />
+          filename="package://priv2/src/priv2_description/meshes/axis_b.STL" />
+      </geometry>
+      <material
+        name="">
+        <color
+          rgba="0.79216 0.81961 0.93333 1" />
+      </material>
+    </visual>
+    <collision>
+      <origin
+        xyz="0 0 0"
+        rpy="0 0 0" />
+      <geometry>
+        <mesh
+          filename="package://priv2/src/priv2_description/meshes/axis_b.STL" />
+      </geometry>
+    </collision>
   </link>
   <joint
@@ -235,6 +194,6 @@
     type="continuous">
     <origin
-      xyz="0.025024 -4.1596E-05 0.002"
-      rpy="-1.5708 0 2.5198" />
+      xyz="0.025024 0 0"
+      rpy="0 0 0" />
     <parent
       link="base_link" />
@@ -242,5 +201,5 @@
       link="wheel_b_axis" />
     <axis
-      xyz="0 1 0" />
+      xyz="0 0 1" />
     <dynamics
       friction="0.002" />
@@ -250,9 +209,9 @@
     <inertial>
       <origin
-        xyz="0 0 0"
-        rpy="0 0 0" />
-      <mass
-        value="0.05" />
-      <inertia
+        xyz="0 -0.0009 0"
+        rpy="0 0 0" />
+      <mass
+        value="0.1" />
+   <inertia
         ixx="4.3881E-08"
         ixy="0"
@@ -285,4 +244,6 @@
       </geometry>
     </collision>
+ <dynamics
+      friction="0.8" />
   </link>
   <joint
@@ -290,6 +251,6 @@
     type="continuous">
     <origin
-      xyz="0 0 0"
-      rpy="-2.7485 0.94901 0" />
+      xyz="0 -0.0009 0.002"
+      rpy="0 0 1.5708" />
     <parent
       link="wheel_b_axis" />

Commit message: Add files via upload

File: priv2/src/priv2_description/urdf/priv2.xacro (robot description, xacro)
@@ -4,4 +4,10 @@
   <xacro:include filename="$(find priv2)/src/priv2_description/urdf/materials.xacro" />
   <xacro:include filename="$(find priv2)/src/priv2_description/urdf/macros.xacro" />
+  <link name="base_footprint"/>
+  <joint name="base_joint" type="fixed">
+    <parent link="base_footprint"/>
+    <child link="base_link"/>
+    <origin xyz="0.0 0.0 0.0" rpy="0 0 0"/>
+  </joint>
  <link  name="base_link">
     <inertial>
@@ -21,5 +27,5 @@
       <origin
         xyz="0 0 0"
-        rpy="0 0 0" /> <!--0.01 0.1 -0.0025 -->
+        rpy="0 0 0" />
       <geometry>
         <mesh
@@ -50,15 +56,15 @@
         value="0.5" />
       <inertia
-        ixx="5.42E-05"
-        ixy="0"
-        ixz="0"
-        iyy="5.42E-05"
-        iyz="0"
-        izz="0.0001" />
-    </inertial>
-    <visual>
-      <origin
-        xyz="0 0 0"
-        rpy="1.57 0 0" /> <!-- 0.0375 0.0175 0.07-->
+        ixx="5.42E-06"
+        ixy="0"
+        ixz="0"
+        iyy="5.42E-06"
+        iyz="0"
+        izz="0.00001" />
+    </inertial>
+    <visual>
+      <origin
+        xyz="0 0 0"
+        rpy="1.57 0 0" />
       <geometry>
         <mesh
@@ -66,7 +72,5 @@
       </geometry>
       <material
-        name="">
-        <color
-          rgba="0.79216 0.81961 0.93333 1" />
+        name="brown">
       </material>
     </visual>
@@ -80,6 +84,4 @@
       </geometry>
     </collision>
- <dynamics
-      friction="1.4" />
   </link>
    <joint
@@ -104,10 +106,10 @@
         value="0.5" />
       <inertia
-        ixx="5.42E-05"
-        ixy="0"
-        ixz="0"
-        iyy="5.42E-05"
-        iyz="0"
-        izz="0.0001" />
+        ixx="5.42E-06"
+        ixy="0"
+        ixz="0"
+        iyy="5.42E-06"
+        iyz="0"
+        izz="0.00001" />
     </inertial>
     <visual>
@@ -134,6 +136,4 @@
       </geometry>
     </collision>
- <dynamics
-      friction="1.4" />
   </link>
   <joint
@@ -202,6 +202,4 @@
     <axis
       xyz="0 0 1" />
-    <dynamics
-      friction="0.002" />
   </joint>
   <link
@@ -244,6 +242,4 @@
       </geometry>
     </collision>
- <dynamics
-      friction="0.8" />
   </link>
   <joint
@@ -251,5 +247,5 @@
     type="continuous">
     <origin
-      xyz="0 -0.0009 0.002"
+      xyz="0.007 -0.0009 0.002"
       rpy="0 0 1.5708" />
     <parent
@@ -260,3 +256,29 @@
       xyz="1 0 0" />
   </joint>
+ <!-- hokuyo -->
+  <link name="hokuyo">
+    <collision>
+      <origin xyz="0 0 0" rpy="0 0 0"/>
+      <geometry>
+    <box size="0.01 0.01 0.01"/>
+      </geometry>
+    </collision>
+    <visual>
+      <origin xyz="0 0 0" rpy="0 0 0"/>
+      <geometry>
+        <mesh filename="package://priv2/src/priv2_description/meshes/hokuyo.dae" scale="0.1 0.1 0.1"/>
+      </geometry>
+    </visual>
+    <inertial>
+      <mass value="1e-5" />
+      <origin xyz="0 0 0" rpy="0 0 0"/>
+      <inertia ixx="1e-6" ixy="0" ixz="0" iyy="1e-6" iyz="0" izz="1e-6" />
+    </inertial>
+  </link>
+    <joint name="hokuyo_joint" type="fixed">
+    <axis xyz="0 1 0" />
+    <origin xyz="-0.04 0 0.0295" rpy="0 0 3.14"/>
+    <parent link="base_link"/>
+    <child link="hokuyo"/>
+  </joint>
 </robot>

Commit message: Add files via upload

File: priv2/src/priv2_description/urdf/priv2.xacro (robot description, xacro)
@@ -8,5 +8,5 @@
     <parent link="base_footprint"/>
     <child link="base_link"/>
-    <origin xyz="0.0 0.0 0.0" rpy="0 0 0"/>
+    <origin xyz="0.0 0.0 0.0" rpy="0 0 3.14"/>
   </joint>
  <link  name="base_link">
@@ -75,19 +75,16 @@
       </material>
     </visual>
-    <collision>
-      <origin
-        xyz="0 0 0"
-        rpy="1.57 0 0" />
-      <geometry>
-        <mesh
-          filename="package://priv2/src/priv2_description/meshes/wheel_r.STL" />
+   <collision>
+       <origin xyz="0 0 0.005" rpy="0 0 0"/>
+      <geometry>
+        <cylinder length="0.01" radius="0.02"/>
       </geometry>
     </collision>
   </link>
    <joint
-    name="Joint_wheel_r"
+    name="joint_wheel_r"
     type="continuous">
     <origin
-      xyz="-0.025 0.03 0.015"
+      xyz="-0.025 0.035 0.015"
       rpy="-1.5708 0 0" />
     <parent
@@ -127,19 +124,16 @@
       </material>
     </visual>
-    <collision>
-      <origin
-        xyz="0 0 0"
-        rpy="1.57 0 0" />
-      <geometry>
-        <mesh
-          filename="package://priv2/src/priv2_description/meshes/wheel_l.STL" />
+  <collision>
+       <origin xyz="0 0 0.005" rpy="0 0 0"/>
+      <geometry>
+        <cylinder length="0.01" radius="0.02"/>
       </geometry>
     </collision>
   </link>
   <joint
-    name="Joint_wheel_l"
+    name="joint_wheel_l"
     type="continuous">
    <origin
-      xyz="-0.025 -0.03 0.015"
+      xyz="-0.025 -0.035 0.015"
       rpy="1.5708 0 0" />
     <parent
@@ -150,5 +144,5 @@
       xyz="0 0 1" />
   </joint>
- <link
+ <!--<link
     name="wheel_b_axis">
     <inertial>
@@ -189,17 +183,17 @@
       </geometry>
     </collision>
-  </link>
+  </link> -->
   <joint
     name="Joint_wheel_b"
     type="continuous">
     <origin
-      xyz="0.025024 0 0"
-      rpy="0 0 0" />
+      xyz="0.025024 0 -0.001"
+      rpy="0 0 1.57" />
     <parent
       link="base_link" />
     <child
-      link="wheel_b_axis" />
-    <axis
-      xyz="0 0 -1" />
+      link="wheel_b" />
+    <axis
+      xyz="1 0 0" />
   </joint>
   <link
@@ -207,5 +201,5 @@
     <inertial>
       <origin
-        xyz="0 -0.0009 0"
+        xyz="0 0 0"
         rpy="0 0 0" />
       <mass
@@ -225,28 +219,30 @@
       <geometry>
         <mesh
-          filename="package://priv2/src/priv2_description/meshes/wheel_b.STL" />
-      </geometry>
-      <material
-        name="">
-        <color
-          rgba="0.79216 0.81961 0.93333 1" />
-      </material>
-    </visual>
-    <collision>
-      <origin
-        xyz="0 0 0"
-        rpy="0 0 0" />
-      <geometry>
-        <mesh
-          filename="package://priv2/src/priv2_description/meshes/wheel_b.STL" />
-      </geometry>
-    </collision>
-  </link>
-  <joint
+          filename="package://priv2/src/priv2_description/meshes/wheel_b.STL"
+	  scale="0.5 0.5 0.5" />
+      </geometry>
+      <material
+        name="">
+        <color
+          rgba="0.79216 0.81961 0.93333 1" />
+      </material>
+    </visual>
+    <collision>
+      <origin
+        xyz="0 0 0"
+        rpy="0 0 0" />
+      <geometry>
+        <mesh
+          filename="package://priv2/src/priv2_description/meshes/wheel_b.STL"
+	scale="0.5 0.5 0.5" />
+      </geometry>
+    </collision>
+  </link>
+ <!-- <joint
     name="Joint_wheel_b_axis"
     type="continuous">
     <origin
-      xyz="0 -0.0009 0.002"
-      rpy="0 0 1.5708" /> <!--007-->
+      xyz="0.0055 -0.0003 -0.0015"
+      rpy="0 0 1.5708" /> 007
     <parent
       link="wheel_b_axis" />
@@ -255,5 +251,5 @@
     <axis
       xyz="1 0 0" />
-  </joint>
+  </joint> -->
  <!-- hokuyo -->
   <link name="hokuyo">

Commit message: Add files via upload

File: priv2/src/priv2_description/urdf/priv2.xacro (robot description, xacro)
@@ -8,10 +8,10 @@
     <parent link="base_footprint"/>
     <child link="base_link"/>
-    <origin xyz="0.0 0.0 0.0" rpy="0 0 3.14"/>
+    <origin xyz="0.0 0.0 0.0" rpy="0 0 0"/>
   </joint>
  <link  name="base_link">
     <inertial>
       <origin
-        xyz="-0.025 0 0"
+        xyz="0.025 0 0"
         rpy="0 0 0" />
       <mass      value="1" />
@@ -27,5 +27,5 @@
       <origin
         xyz="0 0 0"
-        rpy="0 0 0" />
+        rpy="0 0 3.14" />
       <geometry>
         <mesh
@@ -41,5 +41,5 @@
       <origin
         xyz="0 0 0"
-        rpy="0 0 0" />
+        rpy="0 0 3.14" />
       <geometry>
         <mesh
@@ -48,5 +48,5 @@
     </collision>
   </link>
- <link   name="wheel_r">
+ <link   name="wheel_l">
     <inertial>
       <origin
@@ -65,5 +65,5 @@
     <visual>
       <origin
-        xyz="0 0 0"
+        xyz="0 0 0.0"
         rpy="1.57 0 0" />
       <geometry>
@@ -86,6 +86,55 @@
     type="continuous">
     <origin
-      xyz="-0.025 0.035 0.015"
-      rpy="-1.5708 0 0" />
+      xyz="0.025 0.035 0.015"
+      rpy="-1.57 0 0" />
+    <parent
+      link="base_link" />
+    <child
+      link="wheel_l" />
+    <axis
+      xyz="0 0 1" />
+  </joint>
+  <link   name="wheel_r">
+    <inertial>
+      <origin
+        xyz="0 0 0"
+        rpy="0 0 0" />
+      <mass
+        value="0.5" />
+      <inertia
+        ixx="5.42E-06"
+        ixy="0"
+        ixz="0"
+        iyy="5.42E-06"
+        iyz="0"
+        izz="0.00001" />
+    </inertial>
+    <visual>
+      <origin
+        xyz="0 0 0"
+        rpy="1.57 3.14 0" /> <!--0.0375 -0.0175 -0.13 -->
+      <geometry>
+        <mesh
+          filename="package://priv2/src/priv2_description/meshes/wheel_l.STL" />
+      </geometry>
+      <material
+        name="">
+        <color
+          rgba="0.79216 0.81961 0.93333 1" />
+      </material>
+    </visual>
+  <collision>
+       <origin xyz="0 0 -0.005" rpy="0 0 0"/>
+      <geometry>
+        <cylinder length="0.01" radius="0.02"/>
+      </geometry>
+    </collision>
+  </link>
+  <joint
+    name="joint_wheel_l"
+    type="continuous">
+   <origin
+      xyz="0.025 -0.035 0.015"
+      rpy="-1.57 0 0" />
     <parent
       link="base_link" />
@@ -95,99 +144,10 @@
       xyz="0 0 1" />
   </joint>
-  <link   name="wheel_l">
-    <inertial>
-      <origin
-        xyz="0 0 0"
-        rpy="0 0 0" />
-      <mass
-        value="0.5" />
-      <inertia
-        ixx="5.42E-06"
-        ixy="0"
-        ixz="0"
-        iyy="5.42E-06"
-        iyz="0"
-        izz="0.00001" />
-    </inertial>
-    <visual>
-      <origin
-        xyz="0 0 0"
-        rpy="1.57 0 0" /> <!--0.0375 -0.0175 -0.13 -->
-      <geometry>
-        <mesh
-          filename="package://priv2/src/priv2_description/meshes/wheel_l.STL" />
-      </geometry>
-      <material
-        name="">
-        <color
-          rgba="0.79216 0.81961 0.93333 1" />
-      </material>
-    </visual>
-  <collision>
-       <origin xyz="0 0 0.005" rpy="0 0 0"/>
-      <geometry>
-        <cylinder length="0.01" radius="0.02"/>
-      </geometry>
-    </collision>
-  </link>
-  <joint
-    name="joint_wheel_l"
-    type="continuous">
-   <origin
-      xyz="-0.025 -0.035 0.015"
-      rpy="1.5708 0 0" />
-    <parent
-      link="base_link" />
-    <child
-      link="wheel_l" />
-    <axis
-      xyz="0 0 1" />
-  </joint>
- <!--<link
-    name="wheel_b_axis">
-    <inertial>
-      <origin
-        xyz="-3.4694E-18 -0.0035 -1.7347E-18"
-        rpy="0 0 0" />
-      <mass
-        value="0.5" />
-      <inertia
-        ixx="2.7941E-08"
-        ixy="0"
-        ixz="0"
-        iyy="4.6383E-08"
-        iyz="0"
-        izz="2.3027E-08" />
-    </inertial>
-    <visual>
-      <origin
-        xyz="0 0 0"
-        rpy="0 0 0" />
-      <geometry>
-        <mesh
-          filename="package://priv2/src/priv2_description/meshes/axis_b.STL" />
-      </geometry>
-      <material
-        name="">
-        <color
-          rgba="0.79216 0.81961 0.93333 1" />
-      </material>
-    </visual>
-    <collision>
-      <origin
-        xyz="0 0 0"
-        rpy="0 0 0" />
-      <geometry>
-        <mesh
-          filename="package://priv2/src/priv2_description/meshes/axis_b.STL" />
-      </geometry>
-    </collision>
-  </link> -->
   <joint
     name="Joint_wheel_b"
     type="continuous">
     <origin
-      xyz="0.025024 0 -0.001"
-      rpy="0 0 1.57" />
+      xyz="-0.025024 0 -0.001"
+      rpy="-1.57 0 0" />
     <parent
       link="base_link" />
@@ -195,5 +155,5 @@
       link="wheel_b" />
     <axis
-      xyz="1 0 0" />
+      xyz="0 0 1" />
   </joint>
   <link
@@ -216,5 +176,5 @@
       <origin
         xyz="0 0 0"
-        rpy="0 0 0" />
+        rpy="0 1.57 0" />
       <geometry>
         <mesh
@@ -231,5 +191,5 @@
       <origin
         xyz="0 0 0"
-        rpy="0 0 0" />
+        rpy="0 1.57 0" />
       <geometry>
         <mesh
@@ -239,17 +199,4 @@
     </collision>
   </link>
- <!-- <joint
-    name="Joint_wheel_b_axis"
-    type="continuous">
-    <origin
-      xyz="0.0055 -0.0003 -0.0015"
-      rpy="0 0 1.5708" /> 007
-    <parent
-      link="wheel_b_axis" />
-    <child
-      link="wheel_b" />
-    <axis
-      xyz="1 0 0" />
-  </joint> -->
  <!-- hokuyo -->
   <link name="hokuyo">
@@ -274,5 +221,5 @@
     <joint name="hokuyo_joint" type="fixed">
     <axis xyz="0 1 0" />
-    <origin xyz="-0.04 0 0.0295" rpy="0 0 3.14"/>
+    <origin xyz="0.04 0 0.0295" rpy="0 0 0"/>
     <parent link="base_link"/>
     <child link="hokuyo"/>
