Commit message: Add files via upload

File: priv2m/priv2_description/urdf/priv2.xacro (robot description, xacro)
@@ -1,8 +1,8 @@
 <?xml version="1.0" encoding="utf-8"?>
-<robot name="priv2" xmlns:xacro="http://www.ros.org/wiki/xacro">
+<robot name="priv2m" xmlns:xacro="http://www.ros.org/wiki/xacro">
   <xacro:arg name="prefix" default=""/>
-  <xacro:include filename="$(find priv2)/priv2_description/urdf/priv2.gazebo" />
-  <xacro:include filename="$(find priv2)/priv2_description/urdf/materials.xacro" />
-  <xacro:include filename="$(find priv2)/priv2_description/urdf/macros.xacro" />
+  <xacro:include filename="$(find priv2m)/priv2_description/urdf/priv2.gazebo" />
+  <xacro:include filename="$(find priv2m)/priv2_description/urdf/materials.xacro" />
+  <xacro:include filename="$(find priv2m)/priv2_description/urdf/macros.xacro" />
   <link name="$(arg prefix)base_footprint"/>
   <joint name="base_joint" type="fixed">
@@ -31,5 +31,5 @@
       <geometry>
         <mesh
-          filename="package://priv2/priv2_description/meshes/base_link.STL" />
+          filename="package://priv2m/priv2_description/meshes/base_link.STL" />
       </geometry>
       <material
@@ -45,5 +45,5 @@
       <geometry>
         <mesh
-          filename="package://priv2/priv2_description/meshes/base_link.STL" />
+          filename="package://priv2m/priv2_description/meshes/base_link.STL" />
       </geometry>
     </collision>
@@ -70,5 +70,5 @@
       <geometry>
         <mesh
-          filename="package://priv2/priv2_description/meshes/wheel_r.STL" />
+          filename="package://priv2m/priv2_description/meshes/wheel_r.STL" />
       </geometry>
       <material
@@ -117,5 +117,5 @@
       <geometry>
         <mesh
-          filename="package://priv2/priv2_description/meshes/wheel_l.STL" />
+          filename="package://priv2m/priv2_description/meshes/wheel_l.STL" />
       </geometry>
       <material
@@ -166,5 +166,5 @@
       <geometry>
         <mesh
-          filename="package://priv2/priv2_description/meshes/wheel_b.STL"
+          filename="package://priv2m/priv2_description/meshes/wheel_b.STL"
 	  scale="0.5 0.5 0.5" />
       </geometry>
@@ -181,5 +181,5 @@
       <geometry>
         <mesh
-          filename="package://priv2/priv2_description/meshes/wheel_b.STL"
+          filename="package://priv2m/priv2_description/meshes/wheel_b.STL"
 	scale="0.5 0.5 0.5" />
       </geometry>
@@ -210,5 +210,5 @@
       <origin xyz="0 0 0" rpy="0 0 0"/>
       <geometry>
-        <mesh filename="package://priv2/priv2_description/meshes/hokuyo.dae" scale="0.1 0.1 0.1"/>
+        <mesh filename="package://priv2m/priv2_description/meshes/hokuyo.dae" scale="0.1 0.1 0.1"/>
       </geometry>
     </visual>
