Commit message: Add files via upload

File: priv2m/priv2_description/urdf/priv2.gazebo.xacro (robot description, xacro)
@@ -7,5 +7,4 @@
       <alwaysOn>false</alwaysOn>
       <updateRate>5</updateRate>
-      <robotNamespace>$(arg prefix)</robotNamespace>
       <leftJoint>joint_wheel_r</leftJoint>
       <rightJoint>joint_wheel_l</rightJoint>
@@ -49,6 +48,14 @@
     <material>Gazebo/FlatBlack</material>
   </gazebo>
-<gazebo reference="$(arg prefix)wheel_b">
+  <gazebo reference="$(arg prefix)wheel_b">
+    <mu1>0.02</mu1>
+    <mu2>0.01</mu2>
+    <kp>500000.0</kp>
+    <kd>10.0</kd>
+    <minDepth>0.0001</minDepth>
+    <maxVel>0.7</maxVel>
+    <fdir1>1 0 0</fdir1>
     <material>Gazebo/FlatBlack</material>
+    <selfCollide>false</selfCollide>
   </gazebo>
  <!-- hokuyo -->
@@ -85,5 +92,4 @@
         <topicName>/priv2/laser/scan</topicName>
         <frameName>hokuyo</frameName>
-        <robotNamespace>$(arg prefix)</robotNamespace>
       </plugin>
     </sensor>

File: priv2m/priv2_description/urdf/priv2.xacro (robot description, xacro)
@@ -114,5 +114,5 @@
       <origin
         xyz="0 0 0"
-        rpy="1.57 3.14 0" /> <!--0.0375 -0.0175 -0.13 -->
+        rpy="1.57 3.14 0" />
       <geometry>
         <mesh
@@ -145,5 +145,31 @@
       xyz="0 0 1" />
   </joint>
-  <link   name="$(arg prefix)wheel_b">
+  <!--<link name="$(arg prefix)test" >
+    <visual>
+       <geometry>
+          <box size="0.01 0.01 0.01"/>
+       </geometry>
+    </visual>
+    <collision>
+       <origin xyz="0 0 -0.005" rpy="0 0 0"/>
+         <geometry>
+            <box size="0.01 0.01 0.01"/>
+         </geometry>
+    </collision>
+  </link>
+  <joint
+    name="$(arg prefix)joint_test"
+    type="fixed">
+    <origin
+      xyz="0 0.01 0"
+      rpy="-1.57 0 0" />
+    <parent
+      link="$(arg prefix)base_link" />
+    <child
+      link="$(arg prefix)test" />
+    <axis
+      xyz="0 0 1" />
+  </joint> -->
+  <link name="$(arg prefix)wheel_b">
     <inertial>
       <origin
@@ -161,35 +187,30 @@
     </inertial>
     <visual>
-      <origin
+        <origin
         xyz="0 0 0"
         rpy="0 1.57 0" />
-      <geometry>
-        <mesh
-          filename="package://priv2m/priv2_description/meshes/wheel_b.STL"
-	  scale="0.5 0.5 0.5" />
-      </geometry>
-      <material
+        <geometry>
+            <cylinder length="0.01" radius="0.0035"/>
+        </geometry>
+        <material
         name="">
-        <color
-          rgba="0.79216 0.81961 0.93333 1" />
-      </material>
-    </visual>
-    <collision>
-      <origin
+          <color rgba="0.79216 0.81961 0.93333 1" />
+        </material>
+    </visual>
+    <collision>
+       <origin
         xyz="0 0 0"
         rpy="0 1.57 0" />
-      <geometry>
-        <mesh
-          filename="package://priv2m/priv2_description/meshes/wheel_b.STL"
-	scale="0.5 0.5 0.5" />
-      </geometry>
+       <geometry>
+          <cylinder length="0.015" radius="0.025"/>
+       </geometry>
     </collision>
   </link>
   <joint
-    name="Joint_wheel_b"
-    type="continuous">
+    name="joint_wheel_b"
+    type="fixed">
     <origin
       xyz="-0.025024 0 -0.001"
-      rpy="-1.57 0 0" />
+      rpy="0 0 1.57" />
     <parent
       link="$(arg prefix)base_link" />

Commit message: Add files via upload

File: priv2m/priv2_description/urdf/priv2.gazebo.xacro (robot description, xacro)
@@ -49,6 +49,6 @@
   </gazebo>
   <gazebo reference="$(arg prefix)wheel_b">
-    <mu1>0.02</mu1>
-    <mu2>0.01</mu2>
+    <mu1>0.001</mu1>
+    <mu2>0.001</mu2>
     <kp>500000.0</kp>
     <kd>10.0</kd>

File: priv2m/priv2_description/urdf/priv2.xacro (robot description, xacro)
@@ -203,5 +203,5 @@
         rpy="0 1.57 0" />
        <geometry>
-          <cylinder length="0.015" radius="0.025"/>
+          <cylinder length="0.01" radius="0.0035"/>
        </geometry>
     </collision>
